File: power_supply_36v_analog/control_driver.kicad_sch (KiCad schematic)
At the start: 38 parts, among them Q5 BC559C, U1 LM723, U2 LM741, U3 LM741

Commit message: Convert global labels to hierarchical pins in all schematic sheets
- control_driver.kicad_sch: US-, output_U-, to_base_driver_adjust, NODO_001, U-
- pwr_driver_output.kicad_sch: AMPERIMETRO+, to_base_driver_adjust, NODO_001, U+
- output_pwr.kicad_sch: U+, V-, U-, output_U-
- power_supply_36v.kicad_sch: TR21, +36V, TR11, TR12, TR22, -36V
- Added corresponding pins to sheet symbols in root schematic
- Updated .gitignore to exclude .history and .lck files
Changed lines of the file:
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@@
     (effects (font (size 1.27 1.27)) (justify left bottom))
   )
-  (global_label "US-" (shape input) (at 177.673 133.35 180) (fields_autoplaced)
-    (effects (font (size 1.27 1.27)) (justify right))
-    (property "Intersheetrefs" "${INTERSHEET_REFS}" (at 170.6548 133.35 0)
-      (effects (font (size 1.27 1.27)) (justify right) hide)
-    )
-  )
-  (global_label "output_U-" (shape input) (at 208.788 151.384 0) (fields_autoplaced)
-    (effects (font (size 1.27 1.27)) (justify left))
-    (property "Intersheetrefs" "${INTERSHEET_REFS}" (at 221.6117 151.384 0)
-      (effects (font (size 1.27 1.27)) (justify left) hide)
-    )
-  )
-  (global_label "to_base_driver_adjust" (shape input) (at 151.765 43.18 0) (fields_autoplaced)
-    (effects (font (size 1.27 1.27)) (justify left))
-    (property "Intersheetrefs" "${INTERSHEET_REFS}" (at 175.051 43.18 0)
-      (effects (font (size 1.27 1.27)) (justify left) hide)
-    )
-  )
-  (global_label "NODO_001" (shape input) (at 189.23 126.492 0) (fields_autoplaced)
-    (effects (font (size 1.27 1.27)) (justify left))
-    (property "Intersheetrefs" "${INTERSHEET_REFS}" (at 201.9934 126.492 0)
-      (effects (font (size 1.27 1.27)) (justify left) hide)
-    )
-  )
-  (global_label "U-" (shape input) (at 209.042 145.288 0) (fields_autoplaced)
-    (effects (font (size 1.27 1.27)) (justify left))
-    (property "Intersheetrefs" "${INTERSHEET_REFS}" (at 214.8507 145.288 0)
-      (effects (font (size 1.27 1.27)) (justify left) hide)
-    )
-  )
-  (global_label "US-" (shape input) (at 114.173 108.458 180) (fields_autoplaced)
-    (effects (font (size 1.27 1.27)) (justify right))
-    (property "Intersheetrefs" "${INTERSHEET_REFS}" (at 107.1548 108.458 0)
-      (effects (font (size 1.27 1.27)) (justify right) hide)
-    )
-  )
+  (hierarchical_label "US-" (shape input) (at 177.673 133.35 180) (effects (font (size 1.27 1.27))))
+  (hierarchical_label "output_U-" (shape input) (at 208.788 151.384 0) (effects (font (size 1.27 1.27))))
+  (hierarchical_label "to_base_driver_adjust" (shape input) (at 151.765 43.18 0) (effects (font (size 1.27 1.27))))
+  (hierarchical_label "NODO_001" (shape input) (at 189.23 126.492 0) (effects (font (size 1.27 1.27))))
+  (hierarchical_label "U-" (shape input) (at 209.042 145.288 0) (effects (font (size 1.27 1.27))))
+  (hierarchical_label "US-" (shape input) (at 114.173 108.458 180) (effects (font (size 1.27 1.27))))
   (netclass_flag "" (length 2.54) (shape round) (at 129.794 77.343 0) (fields_autoplaced)
     (effects (font (size 1.27 1.27)) (justify left bottom))

Commit message: Fix pin spacing to 2.54mm like DiscoveryAnalog3 sheet
Parts:
- renumbered C3 to C403, C4 to C404, C6 to C405, C7 to C406, C8 to C407, C9 to C408, D9 to D401, D11 to D402, D12 to D403, D13 to D404, D14 to D405, DZ1 to DZ401, LED1 to LED401, Q5 to Q401, R1 to R401, R2 to R402, R3 to R403, R4 to R404, R5 to R405, R6 to R406, R7 to R407, R8 to R408, R9 to R409, R11 to R410, R17 to R411, R101 to R412, R18 to R413, R19 to R414, R20 to R415, R21 to R416, R23 to R417, R25 to R418, R24 to R419, RV4 to RV401, RV3 to RV402, U1 to U401, U2 to U402, U3 to U403
