File: power_supply_36v_analog/power_supply_36v.kicad_sch (KiCad schematic)
At the start: 15 parts, among them J1 Transformador 15 + 15 volt AC, J2 Transformador 36 volt AC

Commit message: Convert global labels to hierarchical pins in all schematic sheets
- control_driver.kicad_sch: US-, output_U-, to_base_driver_adjust, NODO_001, U-
- pwr_driver_output.kicad_sch: AMPERIMETRO+, to_base_driver_adjust, NODO_001, U+
- output_pwr.kicad_sch: U+, V-, U-, output_U-
- power_supply_36v.kicad_sch: TR21, +36V, TR11, TR12, TR22, -36V
- Added corresponding pins to sheet symbols in root schematic
- Updated .gitignore to exclude .history and .lck files
Changed lines of the file:
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@@
     (stroke (width 0) (type default))
   )
-  (global_label "TR21" (shape input) (at 72.136 82.296 180) (fields_autoplaced)
-    (effects (font (size 1.27 1.27)) (justify right))
-    (property "Intersheetrefs" "${INTERSHEET_REFS}" (at 64.5736 82.296 0)
-      (effects (font (size 1.27 1.27)) (justify right) hide)
-    )
-  )
-  (global_label "+36V" (shape input) (at 186.055 71.374 0) (fields_autoplaced)
-    (effects (font (size 1.27 1.27)) (justify left))
-    (property "Intersheetrefs" "${INTERSHEET_REFS}" (at 194.0408 71.374 0)
-      (effects (font (size 1.27 1.27)) (justify left) hide)
-    )
-  )
-  (global_label "TR11" (shape input) (at 125.349 133.731 180) (fields_autoplaced)
-    (effects (font (size 1.27 1.27)) (justify right))
-    (property "Intersheetrefs" "${INTERSHEET_REFS}" (at 117.7866 133.731 0)
-      (effects (font (size 1.27 1.27)) (justify right) hide)
-    )
-  )
-  (global_label "TR21" (shape input) (at 114.681 76.327 180) (fields_autoplaced)
-    (effects (font (size 1.27 1.27)) (justify right))
-    (property "Intersheetrefs" "${INTERSHEET_REFS}" (at 107.1186 76.327 0)
-      (effects (font (size 1.27 1.27)) (justify right) hide)
-    )
-  )
-  (global_label "TR12" (shape input) (at 67.31 143.891 180) (fields_autoplaced)
-    (effects (font (size 1.27 1.27)) (justify right))
-    (property "Intersheetrefs" "${INTERSHEET_REFS}" (at 59.7476 143.891 0)
-      (effects (font (size 1.27 1.27)) (justify right) hide)
-    )
-  )
-  (global_label "TR11" (shape input) (at 67.31 138.811 180) (fields_autoplaced)
-    (effects (font (size 1.27 1.27)) (justify right))
-    (property "Intersheetrefs" "${INTERSHEET_REFS}" (at 59.7476 138.811 0)
-      (effects (font (size 1.27 1.27)) (justify right) hide)
-    )
-  )
-  (global_label "TR22" (shape input) (at 72.136 84.836 180) (fields_autoplaced)
-    (effects (font (size 1.27 1.27)) (justify right))
-    (property "Intersheetrefs" "${INTERSHEET_REFS}" (at 64.5736 84.836 0)
-      (effects (font (size 1.27 1.27)) (justify right) hide)
-    )
-  )
-  (global_label "-36V" (shape input) (at 188.468 101.219 0) (fields_autoplaced)
-    (effects (font (size 1.27 1.27)) (justify left))
-    (property "Intersheetrefs" "${INTERSHEET_REFS}" (at 196.4538 101.219 0)
-      (effects (font (size 1.27 1.27)) (justify left) hide)
-    )
-  )
-  (global_label "TR22" (shape input) (at 137.033 96.901 180) (fields_autoplaced)
-    (effects (font (size 1.27 1.27)) (justify right))
-    (property "Intersheetrefs" "${INTERSHEET_REFS}" (at 129.4706 96.901 0)
-      (effects (font (size 1.27 1.27)) (justify right) hide)
-    )
-  )
-  (global_label "TR12" (shape input) (at 125.349 160.401 180) (fields_autoplaced)
-    (effects (font (size 1.27 1.27)) (justify right))
-    (property "Intersheetrefs" "${INTERSHEET_REFS}" (at 117.7866 160.401 0)
-      (effects (font (size 1.27 1.27)) (justify right) hide)
-    )
-  )
+  (hierarchical_label "TR21" (shape input) (at 72.136 82.296 180) (effects (font (size 1.27 1.27))))
+  (hierarchical_label "+36V" (shape input) (at 186.055 71.374 0) (effects (font (size 1.27 1.27))))
+  (hierarchical_label "TR11" (shape input) (at 125.349 133.731 180) (effects (font (size 1.27 1.27))))
+  (hierarchical_label "TR21" (shape input) (at 114.681 76.327 180) (effects (font (size 1.27 1.27))))
+  (hierarchical_label "TR12" (shape input) (at 67.31 143.891 180) (effects (font (size 1.27 1.27))))
+  (hierarchical_label "TR11" (shape input) (at 67.31 138.811 180) (effects (font (size 1.27 1.27))))
+  (hierarchical_label "TR22" (shape input) (at 72.136 84.836 180) (effects (font (size 1.27 1.27))))
+  (hierarchical_label "-36V" (shape input) (at 188.468 101.219 0) (effects (font (size 1.27 1.27))))
+  (hierarchical_label "TR22" (shape input) (at 137.033 96.901 180) (effects (font (size 1.27 1.27))))
+  (hierarchical_label "TR12" (shape input) (at 125.349 160.401 180) (effects (font (size 1.27 1.27))))
   (symbol (lib_id "Library_power_labs_libraries:L") (at 167.005 76.327 90) (unit 1)
     (in_bom yes) (on_board yes) (dnp no)

Commit message: Fix pin spacing to 2.54mm like DiscoveryAnalog3 sheet
Parts:
- renumbered C5 to C201, C1 to C204, C2 to C205, D5 to D201, D6 to D202, D8 to D203, D7 to D204, D1 to D205, D2 to D206, D3 to D207, D4 to D208, J2 to J201, J1 to J202, L1 to L201, L2 to L202
