File: power_supply_36v_analog/pwr_driver_output.kicad_sch (KiCad schematic)
At the start: 15 parts, among them Q1 BD241, Q2 2N3055, Q3 2N3055, Q4 2N3055

Commit message: Convert global labels to hierarchical pins in all schematic sheets
- control_driver.kicad_sch: US-, output_U-, to_base_driver_adjust, NODO_001, U-
- pwr_driver_output.kicad_sch: AMPERIMETRO+, to_base_driver_adjust, NODO_001, U+
- output_pwr.kicad_sch: U+, V-, U-, output_U-
- power_supply_36v.kicad_sch: TR21, +36V, TR11, TR12, TR22, -36V
- Added corresponding pins to sheet symbols in root schematic
- Updated .gitignore to exclude .history and .lck files
Changed lines of the file:
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@@
     (stroke (width 0) (type default))
   )
-  (global_label "AMPERIMETRO+" (shape input) (at 176.657 77.089 180) (fields_autoplaced)
-    (effects (font (size 1.27 1.27)) (justify right))
-    (property "Intersheetrefs" "${INTERSHEET_REFS}" (at 159.1765 77.089 0)
-      (effects (font (size 1.27 1.27)) (justify right) hide)
-    )
-  )
-  (global_label "to_base_driver_adjust" (shape input) (at 109.728 109.093 0) (fields_autoplaced)
-    (effects (font (size 1.27 1.27)) (justify left))
-    (property "Intersheetrefs" "${INTERSHEET_REFS}" (at 133.014 109.093 0)
-      (effects (font (size 1.27 1.27)) (justify left) hide)
-    )
-  )
-  (global_label "NODO_001" (shape input) (at 145.796 65.151 0) (fields_autoplaced)
-    (effects (font (size 1.27 1.27)) (justify left))
-    (property "Intersheetrefs" "${INTERSHEET_REFS}" (at 158.5594 65.151 0)
-      (effects (font (size 1.27 1.27)) (justify left) hide)
-    )
-  )
-  (global_label "U+" (shape input) (at 208.28 72.517 0) (fields_autoplaced)
-    (effects (font (size 1.27 1.27)) (justify left))
-    (property "Intersheetrefs" "${INTERSHEET_REFS}" (at 214.0887 72.517 0)
-      (effects (font (size 1.27 1.27)) (justify left) hide)
-    )
-  )
+  (hierarchical_label "AMPERIMETRO+" (shape input) (at 176.657 77.089 180) (effects (font (size 1.27 1.27))))
+  (hierarchical_label "to_base_driver_adjust" (shape input) (at 109.728 109.093 0) (effects (font (size 1.27 1.27))))
+  (hierarchical_label "NODO_001" (shape input) (at 145.796 65.151 0) (effects (font (size 1.27 1.27))))
+  (hierarchical_label "U+" (shape input) (at 208.28 72.517 0) (effects (font (size 1.27 1.27))))
   (netclass_flag "" (length 2.54) (shape round) (at 194.691 92.202 180) (fields_autoplaced)
     (effects (font (size 1.27 1.27)) (justify right bottom))

Commit message: Fix pin spacing to 2.54mm like DiscoveryAnalog3 sheet
Parts:
- renumbered C10 to C301, D10 to D301, R15 to J301, Q1 to Q301, Q2 to Q302, Q3 to Q303, Q4 to Q304, R10 to R301, R12 to R302, R14 to R303, R13 to R304, R15 to R305, R16 to R306, R22 to R307, RV1 to RV301
